File: PCB/IRHub_PCB_V3/IRHub_V3.kicad_pcb (KiCad board)
At the start: 2 copper layers, 66 parts, among them J2 USB_C_Receptacle_USB2.0_16P, Q1 UMH3N, Q2 AO3400A, Q3 AO3400A, U1 ESP-12F, U2 CH340C, U3 AMS1117-3.3, U4 TSOP382xx, U5 ME6211C33M5

Commit message: complete schematic i think ?
Parts:
- removed OLED1: Conn_01x04_Pin, Connector_PinHeader_2.54mm:PinHeader_1x04_P2.54mm_Vertical
- added 5V1: VCC, TestPoint:TestPoint_Pad_D2.0mm, F.Cu at (141.8, 92.4)
- added J1: DispTouch, Connector_JST:JST_SH_BM06B-SRSS-TB_1x06-1MP_P1.00mm_Vertical, F.Cu at (157.3, 103.5)
- added TP9: 3V3, TestPoint:TestPoint_Pad_D2.0mm, F.Cu at (141.8, 96.4)
- added T_D+1: D+, TestPoint:TestPoint_Pad_D2.0mm, F.Cu at (145.8, 96.4)
- added T_D-1: D-, TestPoint:TestPoint_Pad_D2.0mm, F.Cu at (145.8, 100.5)
- added T_D6: D6, TestPoint:TestPoint_Pad_D2.0mm, F.Cu at (141.8, 100.5)
- added T_D7: D7, TestPoint:TestPoint_Pad_D2.0mm, F.Cu at (145.8, 92.4)
- added T_GND1: GND, TestPoint:TestPoint_Pad_D2.0mm, F.Cu at (149.9, 92.4)
- added T_RX1: RX, TestPoint:TestPoint_Pad_D2.0mm, F.Cu at (149.9, 96.4)
- added T_TX1: TX, TestPoint:TestPoint_Pad_D2.0mm, F.Cu at (149.9, 100.5)
- LS1: footprint CMT-7525-80-SMT-TR:XDCR_CMT-7525-80-SMT-TR -> CMT-7525:XDCR_CMT-7525-80-SMT-TR
- moved U3 43.9 mm to (166.3, 73.9)
- moved U2 37.5 mm to (165.6, 64.0)
- moved U4 31.8 mm to (164.4, 102.5)
- moved LS1 31.6 mm to (172.4, 93.4)
- moved U5 29.8 mm to (142.3, 104.9)
- moved Q1 29.8 mm to (147.0, 104.5)
- moved R1 24.0 mm to (135.3, 86.1)
- moved R2 24.0 mm to (135.3, 89.4)
- moved R3 24.0 mm to (135.3, 92.7)
- moved R4 24.0 mm to (135.3, 96.0)
- moved J2 19.8 mm to (159.1, 95.6)
- moved C3 7.85 mm to (166.3, 81.1)
- moved D11 7.85 mm to (146.2, 74.1)
- moved D23 7.85 mm to (154.9, 74.1)
- moved D29 7.85 mm to (159.2, 74.1)
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